Commit message: pendulum urdf

File: description/robot.urdf.xacro (robot description, xacro)
@@ -77,4 +77,13 @@
             <material name="orange"/>
         </visual>
+        <collision>
+            <origin xyz="0 0 0" rpy="0 0 0"/>
+            <geometry>
+                <cylinder radius="${wheel_radius}" length="${wheel_thickness}"/>
+            </geometry>
+        </collision>
+        <xacro:inertial_cylinder mass="${wheel_mass}" length="${wheel_thickness}" radius="${wheel_radius}">
+            <origin xyz="0 0 0" rpy="0 0 0"/>
+        </xacro:inertial_cylinder>
     </link>
 </robot>

Commit message: sim imu

File: description/robot.urdf.xacro (robot description, xacro)
@@ -2,4 +2,5 @@
 <robot xmlns:xacro="http://www.ros.org/wiki/xacro"  name="robot">
     <xacro:include filename="inertia_tensor.xacro"/>
+    <xacro:include filename="gazebo_control.xacro"/>
     <xacro:property name="arm_length" value="1"/>
     <xacro:property name="arm_width" value="0.1"/>
@@ -9,4 +10,5 @@
     <xacro:property name="wheel_thickness" value="0.02"/>
     <xacro:property name="wheel_mass" value="0.05"/>
+    <xacro:property name="imu_distance" value="0.65"/>
     <link name="world"></link>
     <!-- base -->
@@ -18,7 +20,7 @@
     <link name="base_link">
         <visual>
-            <origin xyz="0 0 0.075" rpy="0 0 0"/>
+            <origin xyz="0 0 0.125" rpy="0 0 0"/>
             <geometry>
-                <box size="0.5 0.25 0.15" />
+                <box size="0.5 0.25 0.25" />
             </geometry>
             <material name="white">
@@ -27,10 +29,10 @@
         </visual>
         <collision>
-            <origin xyz="0 0 0.05" rpy="0 0 0"/>
+            <origin xyz="0 0 0.125" rpy="0 0 0"/>
             <geometry>
-                <box size="0.5 0.25 0.15" />
+                <box size="0.5 0.25 0.25" />
             </geometry>
         </collision>
-        <xacro:inertial_box mass="12" x="0.5" y="0.25" z="0.15">
+        <xacro:inertial_box mass="12" x="0.5" y="0.25" z="0.25">
             <origin xyz="0 0 0.05" rpy="0 0 0"/>
         </xacro:inertial_box>
@@ -64,5 +66,5 @@
     <!-- wheel -->
     <joint name="wheel_joint" type="continuous">
-        <origin xyz="0 0.01 1" rpy="-${pi/2} 0 0"/>
+        <origin xyz="0 0.02 ${arm_length}" rpy="-${pi/2} 0 0"/>
         <parent link="arm_link"/>
         <child link="wheel_link"/>
@@ -87,3 +89,27 @@
         </xacro:inertial_cylinder>
     </link>
+    <!-- imu -->
+    <joint name="imu_joint" type="fixed">
+        <origin xyz="0 0.02 ${imu_distance}" rpy="0 0 0"/>
+        <parent link="arm_link"/>
+        <child link="imu_link"/>
+    </joint>
+    <link name="imu_link">
+        <visual>
+            <origin xyz="0 0 0" rpy="0 0 0"/>
+            <geometry>
+                <box size="${arm_width} 0.02 ${arm_width}"/>
+            </geometry>
+            <material name="white"/>
+        </visual>
+        <collision>
+            <origin xyz="0 0 0" rpy="0 0 0"/>
+            <geometry>
+                <box size="${arm_width} 0.02 ${arm_width}"/>
+            </geometry>
+        </collision>
+        <xacro:inertial_box mass="0.01" x="${arm_width}" y="0.02" z="${arm_width}">
+            <origin xyz="0 0 0" rpy="0 0 0"/>
+        </xacro:inertial_box>
+    </link>
 </robot>

Commit message: motor model

File: description/robot.urdf.xacro (robot description, xacro)
@@ -113,3 +113,27 @@
         </xacro:inertial_box>
     </link>
+    <!-- motor -->
+    <joint name="motor_joint" type="fixed">
+        <origin xyz="0 -0.03 0.95" rpy="0 0 0"/>
+        <parent link="arm_link"/>
+        <child link="motor_link"/>
+    </joint>
+    <link name="motor_link">
+        <visual>
+            <origin xyz="0 0 0" rpy="0 0 0"/>
+            <geometry>
+                <box size="${arm_width} 0.05 ${arm_width}"/>
+            </geometry>
+            <material name="white"/>
+        </visual>
+        <collision>
+            <origin xyz="0 0 0" rpy="0 0 0"/>
+            <geometry>
+                <box size="${arm_width} 0.05 ${arm_width}"/>
+            </geometry>
+        </collision>
+        <xacro:inertial_box mass="0.01" x="${arm_width}" y="0.05" z="${arm_width}">
+            <origin xyz="0 0 0" rpy="0 0 0"/>
+        </xacro:inertial_box>
+    </link>
 </robot>
